File: platine/rfid.pcb.kicad_pcb (KiCad board)
At the start: 2 copper layers, 53 x 55 mm, 10 parts, among them J1 TFT Display, J2 RFID Reader, J3 Conn_01x04_Socket, U2 ESP32-C3_SUPERMINI

Commit message: Änderungen für Dietmar
Connections:
- J3 pad 3: unconnected-(J3-Pin_3-Pad3) -> GND
- U2 pad 1: /SD_CS -> Net-(J3-Pin_4)
- U2 pad 3: Net-(J3-Pin_4) -> /SD_CS
Routing:
- net Net-(J3-Pin_4): track 41.7 -> 37.0 mm
- net /SD_CS: track 97.5 -> 100.1 mm
- net GND: track 91.2 -> 93.8 mm
Other:
- board text added: "Buzzer"
- board text removed: "GP1"
- board text removed: "GP3"
Changed lines of the file:
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@@
 	(net 18 "/3V3")
 	(net 19 "Net-(J3-Pin_4)")
-	(net 20 "unconnected-(J3-Pin_3-Pad3)")
 	(footprint "MountingHole:MountingHole_4mm"
 		(layer "F.Cu")
@@
 			(at 0 10.39 90)
 			(layer "F.Fab")
+			(hide yes)
 			(effects
 				(font
@@
 			)
 		)
-		(property "Datasheet" ""
+		(property "Datasheet" "~"
 			(at 0 0 90)
 			(layer "F.Fab")
@@
 			(layers "*.Cu" "*.Mask")
 			(remove_unused_layers no)
-			(net 20 "unconnected-(J3-Pin_3-Pad3)")
+			(net 6 "GND")
 			(pinfunction "Pin_3")
 			(pintype "passive")
@@
 			(layers "*.Cu" "*.Mask")
 			(remove_unused_layers no)
-			(net 3 "/SD_CS")
+			(net 19 "Net-(J3-Pin_4)")
 			(pinfunction "GPIO1")
 			(pintype "bidirectional")
@@
 			(layers "*.Cu" "*.Mask")
 			(remove_unused_layers no)
-			(net 19 "Net-(J3-Pin_4)")
+			(net 3 "/SD_CS")
 			(pinfunction "GPIO3")
 			(pintype "bidirectional")
@@
 		)
 	)
-	(gr_text "GP1"
+	(gr_text "GND"
 		(at 157 133 90)
 		(layer "B.SilkS")
@@
 		)
 	)
-	(gr_text "GP3"
-		(at 154.5 133 90)
+	(gr_text "Buzzer"
+		(at 154.25 130.25 90)
 		(layer "B.SilkS")
 		(effects
@@
 	)
 	(segment
-		(start 159 120)
-		(end 174.951 135.951)
+		(start 160 106.9)
+		(end 160 119)
 		(width 0.5)
 		(layer "F.Cu")
@@
 	)
 	(segment
-		(start 174.951 135.951)
-		(end 182.549 135.951)
+		(start 177 136)
+		(end 183.25 136)
 		(width 0.5)
 		(layer "F.Cu")
@@
 	)
 	(segment
-		(start 182.549 135.951)
-		(end 191.5 127)
+		(start 160 119)
+		(end 177 136)
 		(width 0.5)
 		(layer "F.Cu")
@@
 	)
 	(segment
-		(start 191.5 127)
-		(end 191.5 125)
-		(width 0.5)
-		(layer "F.Cu")
-		(net 3)
-	)
-	(segment
-		(start 159 108)
-		(end 159 120)
-		(width 0.5)
-		(layer "F.Cu")
-		(net 3)
-	)
-	(segment
-		(start 156.24 105.24)
-		(end 159 108)
-		(width 0.5)
-		(layer "F.Cu")
-		(net 3)
-	)
-	(segment
-		(start 153.26 105.24)
-		(end 156.24 105.24)
+		(start 153.26 100.16)
+		(end 160 106.9)
 		(width 0.5)
 		(layer "F.Cu")
@@
 	)
 	(via
-		(at 191.5 125)
+		(at 183.25 136)
 		(size 0.6)
 		(drill 0.3)
@@
 	)
 	(segment
-		(start 191.5 105)
-		(end 191.5 125)
+		(start 180 99.46)
+		(end 185.96 99.46)
 		(width 0.5)
 		(layer "B.Cu")
@@
 	)
 	(segment
-		(start 180 99.46)
-		(end 185.96 99.46)
+		(start 191.5 127.75)
+		(end 183.25 136)
 		(width 0.5)
 		(layer "B.Cu")
@@
 	)
 	(segment
+		(start 191.5 105)
+		(end 191.5 127.75)
+		(width 0.5)
+		(layer "B.Cu")
+		(net 3)
+	)
+	(segment
 		(start 186.5 106.5)
 		(end 188 105)
@@
 	)
 	(segment
+		(start 155.92 139.5)
+		(end 158.46 139.5)
+		(width 1)
+		(layer "B.Cu")
+		(net 6)
+	)
+	(segment
 		(start 187 120)
 		(end 188.5 120)
@@
 	)
 	(segment
+		(start 161.11 117.11)
+		(end 161 117)
+		(width 0.5)
+		(layer "F.Cu")
+		(net 11)
+	)
+	(segment
+		(start 161 105.36)
+		(end 153.26 97.62)
+		(width 0.5)
+		(layer "F.Cu")
+		(net 11)
+	)
+	(segment
 		(start 181.1 117.24)
 		(end 180 117.24)
@@
 		(net 11)
 	)
-	(segment
-		(start 161 105.36)
-		(end 153.26 97.62)
-		(width 0.5)
-		(layer "F.Cu")
-		(net 11)
-	)
 	(via
-		(at 161 117)
+		(at 161.11 117.11)
 		(size 0.6)
 		(drill 0.3)
@@
 	)
 	(segment
-		(start 161.24 117.24)
-		(end 161 117)
+		(start 161.11 117.11)
+		(end 161.24 117.24)
 		(width 0.5)
 		(layer "B.Cu")
@@
 	)
 	(segment
-		(start 180 117.24)
-		(end 161.24 117.24)
+		(start 161.24 117.24)
+		(end 180 117.24)
 		(width 0.5)
 		(layer "B.Cu")
@@
 	)
 	(segment
-		(start 156.770085 107.78)
+		(start 157.78 107.78)
 		(end 153.26 107.78)
 		(width 0.5)
@@
 	)
 	(segment
-		(start 157.5 120)
-		(end 157.5 108.509915)
+		(start 158 108)
+		(end 157.78 107.78)
 		(width 0.5)
 		(layer "F.Cu")
@@
 	)
 	(segment
-		(start 157.5 108.509915)
-		(end 156.770085 107.78)
+		(start 174.265 136.015)
+		(end 158 119.75)
 		(width 0.5)
 		(layer "F.Cu")
@@
 	)
 	(segment
-		(start 173 135.5)
-		(end 157.5 120)
+		(start 158 119.75)
+		(end 158 108)
 		(width 0.5)
 		(layer "F.Cu")
@@
 	)
 	(via
-		(at 173 135.5)
+		(at 174.265 136.015)
 		(size 0.6)
 		(drill 0.3)
@@
 	)
 	(segment
-		(start 184.5 135.5)
-		(end 190.5 129.5)
+		(start 190.5 127.25)
+		(end 190.5 105.5)
 		(width 0.5)
 		(layer "B.Cu")
@@
 	)
 	(segment
-		(start 190.5 105.5)
-		(end 185.5 100.5)
+		(start 185.5 100.5)
+		(end 181.5 100.5)
 		(width 0.5)
 		(layer "B.Cu")
@@
 	)
 	(segment
-		(start 190.5 129.5)
-		(end 190.5 105.5)
+		(start 175 136.75)
+		(end 181 136.75)
 		(width 0.5)
 		(layer "B.Cu")
@@
 	)
 	(segment
-		(start 173 135.5)
-		(end 184.5 135.5)
+		(start 181 136.75)
+		(end 190.5 127.25)
 		(width 0.5)
 		(layer "B.Cu")
@@
 	)
 	(segment
-		(start 185.5 100.5)
-		(end 181.5 100.5)
+		(start 174.265 136.015)
+		(end 175 136.75)
+		(width 0.5)
+		(layer "B.Cu")
+		(net 12)
+	)
+	(segment
+		(start 190.5 105.5)
+		(end 185.5 100.5)
 		(width 0.5)
 		(layer "B.Cu")
@@
 	)
 	(segment
-		(start 160 119.5)
-		(end 160 106.5)
+		(start 159 107.633637)
+		(end 159 119.25)
 		(width 0.5)
 		(layer "F.Cu")
@@
 	)
 	(segment
-		(start 160 106.5)
-		(end 156.2 102.7)
+		(start 154.066363 102.7)
+		(end 159 107.633637)
 		(width 0.5)
 		(layer "F.Cu")
@@
 	)
 	(segment
-		(start 156.2 102.7)
-		(end 153.26 102.7)
+		(start 159 119.25)
+		(end 175.75 136)
 		(width 0.5)
 		(layer "F.Cu")
@@
 	)
 	(segment
-		(start 175 134.5)
-		(end 160 119.5)
+		(start 153.26 102.7)
+		(end 154.066363 102.7)
 		(width 0.5)
 		(layer "F.Cu")
@@
 	)
 	(via
-		(at 175 134.5)
+		(at 175.75 136)
 		(size 0.6)
 		(drill 0.3)
@@
 	)
 	(via
-		(at 175 134.5)
+		(at 175.75 136)
 		(size 0.6)
 		(drill 0.3)
@@
 	)
 	(segment
-		(start 183 111.5)
-		(end 183 126.5)
+		(start 180 136)
+		(end 175.75 136)
 		(width 0.5)
 		(layer "B.Cu")
@@
 	(segment
 		(start 183 133)
-		(end 181.5 134.5)
+		(end 180 136)
 		(width 0.5)
 		(layer "B.Cu")
@@
 	)
 	(segment
-		(start 186.5 108)
-		(end 183 111.5)
+		(start 183 131.5)
+		(end 183 133)
 		(width 0.5)
 		(layer "B.Cu")
@@
 	)
 	(segment
-		(start 187.2 107.3)
-		(end 186.5 108)
+		(start 183 111.5)
+		(end 183 126.5)
 		(width 0.5)
 		(layer "B.Cu")
@@
 	)
 	(segment
-		(start 181.5 134.5)
-		(end 175 134.5)
+		(start 186.5 108)
+		(end 183 111.5)
 		(width 0.5)
 		(layer "B.Cu")
@@
 	)
 	(segment
-		(start 183 131.5)
-		(end 183 133)
+		(start 187.2 107.3)
+		(end 186.5 108)
 		(width 0.5)
 		(layer "B.Cu")
@@
 	)
 	(segment
-		(start 151.5 101.92)
-		(end 153.26 100.16)
-		(width 0.5)
-		(layer "B.Cu")
-		(net 19)
-	)
-	(segment
-		(start 153.42 139.475)
-		(end 154.5 138.395)
-		(width 0.5)
-		(layer "B.Cu")
-		(net 19)
-	)
-	(segment
-		(start 154.5 138.395)
-		(end 154.5 125)
+		(start 150 136.12)
+		(end 150 108.5)
 		(width 0.5)
 		(layer "B.Cu")
@@
 	)
 	(segment
-		(start 154.5 125)
-		(end 151.5 122)
+		(start 150 108.5)
+		(end 153.26 105.24)
 		(width 0.5)
 		(layer "B.Cu")
@@
 	)
 	(segment
-		(start 151.5 122)
-		(end 151.5 101.92)
+		(start 153.38 139.5)
+		(end 150 136.12)
 		(width 0.5)
 		(layer "B.Cu")
