File: platine/rfid.pcb.kicad_sch (KiCad schematic)
At the start: 4 parts, among them J1 TFT Display, J2 RFID Reader, J3 Conn_01x04_Socket, U2 ESP32-C3_SUPERMINI

Commit message: Änderungen für Dietmar
Connections:
- net GND: now also J3.3 (Pin_3)
- net SD_CS: now also U2.3 (GPIO3); no longer U2.1 (GPIO1)
- net at J3.4 (Pin_4): now also U2.1 (GPIO1); no longer U2.3 (GPIO3)
Other:
- moved on the sheet: J3
Changed lines of the file:
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@@
+	)
+	(junction
+		(at 130.81 128.27)
+		(diameter 0)
+		(color 0 0 0 0)
 	)
 	(junction
@@
 	(wire
 		(pts
-			(xy 109.22 85.09) (xy 121.92 85.09)
-		)
-		(stroke
-			(width 0)
-			(type default)
-		)
-	)
-	(wire
-		(pts
-			(xy 119.38 121.92) (xy 130.81 121.92)
-		)
-		(stroke
-			(width 0)
-			(type default)
-		)
-	)
-	(wire
-		(pts
 			(xy 95.25 77.47) (xy 95.25 86.36)
 		)
@@
 	(wire
 		(pts
+			(xy 105.41 88.9) (xy 105.41 85.09)
+		)
+		(stroke
+			(width 0)
+			(type default)
+		)
+	)
+	(wire
+		(pts
 			(xy 64.77 55.88) (xy 74.93 55.88)
 		)
@@
 	(wire
 		(pts
-			(xy 130.81 127) (xy 121.92 127)
-		)
-		(stroke
-			(width 0)
-			(type default)
-		)
-	)
-	(wire
-		(pts
 			(xy 91.44 96.52) (xy 74.93 96.52)
 		)
@@
 	(wire
 		(pts
-			(xy 121.92 127) (xy 121.92 85.09)
-		)
-		(stroke
-			(width 0)
-			(type default)
-		)
-	)
-	(wire
-		(pts
 			(xy 109.22 57.15) (xy 152.4 57.15)
 		)
@@
 	(wire
 		(pts
+			(xy 127 128.27) (xy 130.81 128.27)
+		)
+		(stroke
+			(width 0)
+			(type default)
+		)
+	)
+	(wire
+		(pts
 			(xy 127 81.28) (xy 127 85.09)
 		)
@@
 	(wire
 		(pts
+			(xy 130.81 128.27) (xy 130.81 130.81)
+		)
+		(stroke
+			(width 0)
+			(type default)
+		)
+	)
+	(wire
+		(pts
 			(xy 129.54 82.55) (xy 129.54 72.39)
 		)
@@
 	(wire
 		(pts
-			(xy 97.79 88.9) (xy 97.79 80.01)
+			(xy 123.19 80.01) (xy 109.22 80.01)
+		)
+		(stroke
+			(width 0)
+			(type default)
+		)
+	)
+	(wire
+		(pts
+			(xy 123.19 133.35) (xy 130.81 133.35)
 		)
 		(stroke
@@
 	(wire
 		(pts
+			(xy 123.19 80.01) (xy 123.19 133.35)
+		)
+		(stroke
+			(width 0)
+			(type default)
+		)
+	)
+	(wire
+		(pts
 			(xy 66.04 71.12) (xy 66.04 92.71)
 		)
@@
 	(wire
 		(pts
+			(xy 105.41 85.09) (xy 109.22 85.09)
+		)
+		(stroke
+			(width 0)
+			(type default)
+		)
+	)
+	(wire
+		(pts
 			(xy 144.78 82.55) (xy 129.54 82.55)
 		)
@@
 	(wire
 		(pts
-			(xy 97.79 80.01) (xy 109.22 80.01)
-		)
-		(stroke
-			(width 0)
-			(type default)
-		)
-	)
-	(wire
-		(pts
 			(xy 120.65 82.55) (xy 120.65 114.3)
 		)
@@
 	(wire
 		(pts
+			(xy 127 129.54) (xy 127 128.27)
+		)
+		(stroke
+			(width 0)
+			(type default)
+		)
+	)
+	(wire
+		(pts
 			(xy 110.49 66.04) (xy 110.49 58.42)
 		)
@@
 	(wire
 		(pts
-			(xy 74.93 88.9) (xy 97.79 88.9)
+			(xy 74.93 88.9) (xy 105.41 88.9)
 		)
 		(stroke
@@
 			)
 			(justify right bottom)
+		)
+	)
+	(symbol
+		(lib_id "power:+5V")
+		(at 130.81 125.73 0)
+		(unit 1)
+		(exclude_from_sim no)
+		(in_bom yes)
+		(on_board yes)
+		(dnp no)
+		(fields_autoplaced yes)
+		(property "Reference" "#PWR07"
+			(at 130.81 129.54 0)
+			(effects
+				(font
+					(size 1.27 1.27)
+				)
+				(hide yes)
+			)
+		)
+		(property "Value" "+5V"
+			(at 130.81 120.65 0)
+			(effects
+				(font
+					(size 1.27 1.27)
+				)
+			)
+		)
+		(property "Footprint" ""
+			(at 130.81 125.73 0)
+			(effects
+				(font
+					(size 1.27 1.27)
+				)
+				(hide yes)
+			)
+		)
+		(property "Datasheet" ""
+			(at 130.81 125.73 0)
+			(effects
+				(font
+					(size 1.27 1.27)
+				)
+				(hide yes)
+			)
+		)
+		(property "Description" "Power symbol creates a global label with name \"+5V\""
+			(at 130.81 125.73 0)
+			(effects
+				(font
+					(size 1.27 1.27)
+				)
+				(hide yes)
+			)
+		)
+		(pin "1"
+		)
+		(instances
+			(project "rfid.pcb"
+				(path "/e4efe8e1-e6b2-46be-a413-aeca04d509bf"
+					(reference "#PWR07")
+					(unit 1)
+				)
+			)
 		)
 	)
@@
 	(symbol
 		(lib_id "power:GND")
-		(at 119.38 121.92 0)
+		(at 127 129.54 0)
 		(unit 1)
 		(exclude_from_sim no)
@@
 		(on_board yes)
 		(dnp no)
-		(fields_autoplaced yes)
 		(property "Reference" "#PWR06"
-			(at 119.38 128.27 0)
+			(at 127 135.89 0)
 			(effects
 				(font
@@
 		)
 		(property "Value" "GND"
-			(at 119.38 127 0)
+			(at 127 134.62 0)
 			(effects
 				(font
@@
 		)
 		(property "Footprint" ""
-			(at 119.38 121.92 0)
+			(at 127 129.54 0)
 			(effects
 				(font
@@
 		)
 		(property "Datasheet" ""
-			(at 119.38 121.92 0)
+			(at 127 129.54 0)
 			(effects
 				(font
@@
 		)
 		(property "Description" "Power symbol creates a global label with name \"GND\" , ground"
-			(at 119.38 121.92 0)
+			(at 127 129.54 0)
 			(effects
 				(font
@@
 				(path "/e4efe8e1-e6b2-46be-a413-aeca04d509bf"
 					(reference "#PWR06")
-					(unit 1)
-				)
-			)
-		)
-	)
-	(symbol
-		(lib_id "power:+5V")
-		(at 130.81 119.38 0)
-		(unit 1)
-		(exclude_from_sim no)
-		(in_bom yes)
-		(on_board yes)
-		(dnp no)
-		(fields_autoplaced yes)
-		(property "Reference" "#PWR07"
-			(at 130.81 123.19 0)
-			(effects
-				(font
-					(size 1.27 1.27)
-				)
-				(hide yes)
-			)
-		)
-		(property "Value" "+5V"
-			(at 130.81 114.3 0)
-			(effects
-				(font
-					(size 1.27 1.27)
-				)
-			)
-		)
-		(property "Footprint" ""
-			(at 130.81 119.38 0)
-			(effects
-				(font
-					(size 1.27 1.27)
-				)
-				(hide yes)
-			)
-		)
-		(property "Datasheet" ""
-			(at 130.81 119.38 0)
-			(effects
-				(font
-					(size 1.27 1.27)
-				)
-				(hide yes)
-			)
-		)
-		(property "Description" "Power symbol creates a global label with name \"+5V\""
-			(at 130.81 119.38 0)
-			(effects
-				(font
-					(size 1.27 1.27)
-				)
-				(hide yes)
-			)
-		)
-		(pin "1"
-		)
-		(instances
-			(project "rfid.pcb"
-				(path "/e4efe8e1-e6b2-46be-a413-aeca04d509bf"
-					(reference "#PWR07")
 					(unit 1)
 				)
@@
 	(symbol
 		(lib_id "Connector:Conn_01x04_Socket")
-		(at 135.89 121.92 0)
+		(at 135.89 128.27 0)
 		(unit 1)
 		(exclude_from_sim no)
@@
 		(fields_autoplaced yes)
 		(property "Reference" "J3"
-			(at 137.16 121.9199 0)
+			(at 137.16 128.2699 0)
 			(effects
 				(font
@@
 		)
 		(property "Value" "Conn_01x04_Socket"
-			(at 137.16 124.4599 0)
+			(at 137.16 130.8099 0)
 			(effects
 				(font
@@
 		)
 		(property "Footprint" "Connector_PinSocket_2.54mm:PinSocket_1x04_P2.54mm_Vertical"
-			(at 135.89 121.92 0)
+			(at 135.89 128.27 0)
 			(effects
 				(font
@@
 		)
 		(property "Datasheet" "~"
-			(at 135.89 121.92 0)
+			(at 135.89 128.27 0)
 			(effects
 				(font
@@
 		)
 		(property "Description" "Generic connector, single row, 01x04, script generated"
-			(at 135.89 121.92 0)
-			(effects
-				(font
+			(at 135.89 128.27 0)
+			(effects
+				(font
